File: Chubut_2/amplifying_channel_custom_bias_tee.kicad_sch (KiCad schematic)
At the start: 6 parts

Commit message: Several updates
Parts:
- removed C12, C16: (no value), symbol Device:C
- added C3, C4, C6, C7: (no value), symbol Device:C
- C5: renamed from C17; value (none) -> 100n; footprint (none) -> Capacitor_SMD:C_0805_2012Metric; Manufacturer (none) -> Samsung Electro-Mechanics; Manufacturer number (none) -> CL05B104KP5NNNC
- L1: value (none) -> L; footprint (none) -> Inductor_SMD:L_0402_1005Metric; Manufacturer (none) -> Taiyo Yuden; Manufacturer number (none) -> BRC2012T1R0M
- L2: value (none) -> L; footprint (none) -> Inductor_SMD:L_0402_1005Metric; Manufacturer (none) -> Murata Electronics; Manufacturer number (none) -> LQW18AN18NG00D
- U2: renamed from U12; value (none) -> PSA4-5043+; footprint (none) -> chubut:MMM1362; Manufacturer (none) -> Mini-Circuits; Manufacturer number (none) -> PSA4-5043+
Connections:
- net 3-5V: now also C3.1
- net GND: now also C3.2, C6.1
- net In: now also C4.1
- net Out: now also C7.2
- net at U2.3 (RF-IN): now also C4.2
- net at L1.2, L2.1: now also C6.2
- net at L2.2, U2.1 (RF-OUT_and_DC-IN): now also C7.1
Other:
- moved on the sheet: C5, L1, L2, U2

Commit message: Removed silkscreen and fixed one track
Parts:
- C12: renamed from C3; value (none) -> 100p; footprint (none) -> Capacitor_SMD:C_0402_1005Metric
- C13: renamed from C4; value (none) -> 1n; footprint (none) -> Capacitor_SMD:C_0402_1005Metric
- C15: renamed from C6; value (none) -> 100p; footprint (none) -> Capacitor_SMD:C_0402_1005Metric
- C16: renamed from C7; value (none) -> 1n; footprint (none) -> Capacitor_SMD:C_0402_1005Metric
- L1: value L -> 2.2µ
- L2: value L -> 18n
- renumbered C5 to C14, U2 to U11
Changed lines of the file:
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@@
   (symbol (lib_id "power:GND") (at 142.748 116.586 0) (unit 1)
     (in_bom yes) (on_board yes) (fields_autoplaced)
-    (property "Reference" "#PWR012" (id 0) (at 142.748 122.936 0)
+    (property "Reference" "#PWR056" (id 0) (at 142.748 122.936 0)
       (effects (font (size 1.27 1.27)) hide)
     )
@@
   (symbol (lib_id "Device:C") (at 105.41 72.136 0) (unit 1)
     (in_bom yes) (on_board yes)
-    (property "Reference" "C3" (id 0) (at 109.474 70.8659 0)
-      (effects (font (size 1.27 1.27)) (justify left))
-    )
-    (property "Value" "" (id 1) (at 109.474 73.4059 0)
-      (effects (font (size 1.27 1.27)) (justify left))
-    )
-    (property "Footprint" "" (id 2) (at 106.3752 75.946 0)
+    (property "Reference" "C12" (id 0) (at 109.474 70.8659 0)
+      (effects (font (size 1.27 1.27)) (justify left))
+    )
+    (property "Value" "100p" (id 1) (at 109.474 73.4059 0)
+      (effects (font (size 1.27 1.27)) (justify left))
+    )
+    (property "Footprint" "Capacitor_SMD:C_0402_1005Metric" (id 2) (at 106.3752 75.946 0)
       (effects (font (size 1.27 1.27)) hide)
     )
@@
   (symbol (lib_id "Device:C") (at 179.324 106.934 90) (unit 1)
     (in_bom yes) (on_board yes)
-    (property "Reference" "C7" (id 0) (at 179.324 99.06 90))
-    (property "Value" "" (id 1) (at 179.324 101.6 90))
-    (property "Footprint" "" (id 2) (at 183.134 105.9688 0)
+    (property "Reference" "C16" (id 0) (at 179.324 99.06 90))
+    (property "Value" "1n" (id 1) (at 179.324 101.6 90))
+    (property "Footprint" "Capacitor_SMD:C_0402_1005Metric" (id 2) (at 183.134 105.9688 0)
       (effects (font (size 1.27 1.27)) hide)
     )
@@
   (symbol (lib_id "Device:C") (at 177.546 85.09 180) (unit 1)
     (in_bom yes) (on_board yes)
-    (property "Reference" "C6" (id 0) (at 173.482 86.3601 0)
-      (effects (font (size 1.27 1.27)) (justify left))
-    )
-    (property "Value" "" (id 1) (at 173.482 83.8201 0)
-      (effects (font (size 1.27 1.27)) (justify left))
-    )
-    (property "Footprint" "" (id 2) (at 176.5808 81.28 0)
+    (property "Reference" "C15" (id 0) (at 173.482 86.3601 0)
+      (effects (font (size 1.27 1.27)) (justify left))
+    )
+    (property "Value" "100p" (id 1) (at 173.482 83.8201 0)
+      (effects (font (size 1.27 1.27)) (justify left))
+    )
+    (property "Footprint" "Capacitor_SMD:C_0402_1005Metric" (id 2) (at 176.5808 81.28 0)
       (effects (font (size 1.27 1.27)) hide)
     )
@@
   (symbol (lib_id "Device:C") (at 130.048 72.136 0) (unit 1)
     (in_bom yes) (on_board yes)
-    (property "Reference" "C5" (id 0) (at 134.112 70.8659 0)
+    (property "Reference" "C14" (id 0) (at 134.112 70.8659 0)
       (effects (font (size 1.27 1.27)) (justify left))
     )
@@
   (symbol (lib_id "power:GND") (at 177.546 88.9 0) (unit 1)
     (in_bom yes) (on_board yes) (fields_autoplaced)
-    (property "Reference" "#PWR013" (id 0) (at 177.546 95.25 0)
-      (effects (font (size 1.27 1.27)) hide)
-    )
-    (property "Value" "" (id 1) (at 177.546 93.726 0))
+    (property "Reference" "#PWR057" (id 0) (at 177.546 95.25 0)
+      (effects (font (size 1.27 1.27)) hide)
+    )
+    (property "Value" "GND" (id 1) (at 177.546 93.726 0))
     (property "Footprint" "" (id 2) (at 177.546 88.9 0)
       (effects (font (size 1.27 1.27)) hide)
@@
       (effects (font (size 1.27 1.27)) (justify left))
     )
-    (property "Value" "L" (id 1) (at 156.464 90.6779 0)
+    (property "Value" "18n" (id 1) (at 156.464 90.6779 0)
       (effects (font (size 1.27 1.27)) (justify left))
     )
@@
   (symbol (lib_id "power:GND") (at 105.41 75.946 0) (unit 1)
     (in_bom yes) (on_board yes) (fields_autoplaced)
-    (property "Reference" "#PWR010" (id 0) (at 105.41 82.296 0)
-      (effects (font (size 1.27 1.27)) hide)
-    )
-    (property "Value" "" (id 1) (at 105.41 80.772 0))
+    (property "Reference" "#PWR054" (id 0) (at 105.41 82.296 0)
+      (effects (font (size 1.27 1.27)) hide)
+    )
+    (property "Value" "GND" (id 1) (at 105.41 80.772 0))
     (property "Footprint" "" (id 2) (at 105.41 75.946 0)
       (effects (font (size 1.27 1.27)) hide)
@@
       (effects (font (size 1.27 1.27)) (justify left))
     )
-    (property "Value" "L" (id 1) (at 156.464 73.4059 0)
+    (property "Value" "2.2µ" (id 1) (at 156.464 73.4059 0)
       (effects (font (size 1.27 1.27)) (justify left))
     )
@@
   (symbol (lib_id "power:GND") (at 130.048 75.946 0) (unit 1)
     (in_bom yes) (on_board yes) (fields_autoplaced)
-    (property "Reference" "#PWR011" (id 0) (at 130.048 82.296 0)
+    (property "Reference" "#PWR055" (id 0) (at 130.048 82.296 0)
       (effects (font (size 1.27 1.27)) hide)
     )
@@
   (symbol (lib_id "Chubut2:PSA4-5043+") (at 142.748 103.124 0) (unit 1)
     (in_bom yes) (on_board yes) (fields_autoplaced)
-    (property "Reference" "U2" (id 0) (at 142.748 99.06 0))
+    (property "Reference" "U11" (id 0) (at 142.748 99.06 0))
     (property "Value" "PSA4-5043+" (id 1) (at 142.748 101.6 0))
     (property "Footprint" "chubut:MMM1362" (id 2) (at 142.748 103.124 0)
@@
   (symbol (lib_id "Device:C") (at 117.094 106.934 90) (unit 1)
     (in_bom yes) (on_board yes)
-    (property "Reference" "C4" (id 0) (at 117.094 99.06 90))
-    (property "Value" "" (id 1) (at 117.094 101.6 90))
-    (property "Footprint" "" (id 2) (at 120.904 105.9688 0)
-      (effects (font (size 1.27 1.27)) hide)
-    )
+    (property "Reference" "C13" (id 0) (at 117.094 99.06 90))
+    (property "Value" "1n" (id 1) (at 117.094 101.6 90))
+    (property "Footprint" "Capacitor_SMD:C_0402_1005Metric" (id 2) (at 120.904 105.9688 0)
+      (effects (font (size 1.27 1.27)) hide)
+    )

Commit message: Added value to 2 inductors that was missing and cleaned up the F.Fab
Parts:
- L1: value 2.2µ -> 1µ
- renumbered C12 to C3, C13 to C4, C14 to C5, C15 to C6, C16 to C7, U11 to U2
Changed lines of the file:
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@@
   (symbol (lib_id "power:GND") (at 142.748 116.586 0) (unit 1)
     (in_bom yes) (on_board yes) (fields_autoplaced)
-    (property "Reference" "#PWR056" (id 0) (at 142.748 122.936 0)
+    (property "Reference" "#PWR012" (id 0) (at 142.748 122.936 0)
       (effects (font (size 1.27 1.27)) hide)
     )
@@
   (symbol (lib_id "Device:C") (at 105.41 72.136 0) (unit 1)
     (in_bom yes) (on_board yes)
-    (property "Reference" "C12" (id 0) (at 109.474 70.8659 0)
+    (property "Reference" "C3" (id 0) (at 109.474 70.8659 0)
       (effects (font (size 1.27 1.27)) (justify left))
     )
@@
   (symbol (lib_id "Device:C") (at 179.324 106.934 90) (unit 1)
     (in_bom yes) (on_board yes)
-    (property "Reference" "C16" (id 0) (at 179.324 99.06 90))
+    (property "Reference" "C7" (id 0) (at 179.324 99.06 90))
     (property "Value" "1n" (id 1) (at 179.324 101.6 90))
     (property "Footprint" "Capacitor_SMD:C_0402_1005Metric" (id 2) (at 183.134 105.9688 0)
@@
   (symbol (lib_id "Device:C") (at 177.546 85.09 180) (unit 1)
     (in_bom yes) (on_board yes)
-    (property "Reference" "C15" (id 0) (at 173.482 86.3601 0)
+    (property "Reference" "C6" (id 0) (at 173.482 86.3601 0)
       (effects (font (size 1.27 1.27)) (justify left))
     )
@@
   (symbol (lib_id "Device:C") (at 130.048 72.136 0) (unit 1)
     (in_bom yes) (on_board yes)
-    (property "Reference" "C14" (id 0) (at 134.112 70.8659 0)
+    (property "Reference" "C5" (id 0) (at 134.112 70.8659 0)
       (effects (font (size 1.27 1.27)) (justify left))
     )
@@
   (symbol (lib_id "power:GND") (at 177.546 88.9 0) (unit 1)
     (in_bom yes) (on_board yes) (fields_autoplaced)
-    (property "Reference" "#PWR057" (id 0) (at 177.546 95.25 0)
+    (property "Reference" "#PWR013" (id 0) (at 177.546 95.25 0)
       (effects (font (size 1.27 1.27)) hide)
     )
@@
   (symbol (lib_id "power:GND") (at 105.41 75.946 0) (unit 1)
     (in_bom yes) (on_board yes) (fields_autoplaced)
-    (property "Reference" "#PWR054" (id 0) (at 105.41 82.296 0)
+    (property "Reference" "#PWR010" (id 0) (at 105.41 82.296 0)
       (effects (font (size 1.27 1.27)) hide)
     )
@@
       (effects (font (size 1.27 1.27)) (justify left))
     )
-    (property "Value" "2.2µ" (id 1) (at 156.464 73.4059 0)
+    (property "Value" "1µ" (id 1) (at 156.464 73.4059 0)
       (effects (font (size 1.27 1.27)) (justify left))
     )
@@
   (symbol (lib_id "power:GND") (at 130.048 75.946 0) (unit 1)
     (in_bom yes) (on_board yes) (fields_autoplaced)
-    (property "Reference" "#PWR055" (id 0) (at 130.048 82.296 0)
+    (property "Reference" "#PWR011" (id 0) (at 130.048 82.296 0)
       (effects (font (size 1.27 1.27)) hide)
     )
@@
   (symbol (lib_id "Chubut2:PSA4-5043+") (at 142.748 103.124 0) (unit 1)
     (in_bom yes) (on_board yes) (fields_autoplaced)
-    (property "Reference" "U11" (id 0) (at 142.748 99.06 0))
+    (property "Reference" "U2" (id 0) (at 142.748 99.06 0))
     (property "Value" "PSA4-5043+" (id 1) (at 142.748 101.6 0))
     (property "Footprint" "chubut:MMM1362" (id 2) (at 142.748 103.124 0)
@@
   (symbol (lib_id "Device:C") (at 117.094 106.934 90) (unit 1)
     (in_bom yes) (on_board yes)
-    (property "Reference" "C13" (id 0) (at 117.094 99.06 90))
+    (property "Reference" "C4" (id 0) (at 117.094 99.06 90))
     (property "Value" "1n" (id 1) (at 117.094 101.6 90))
     (property "Footprint" "Capacitor_SMD:C_0402_1005Metric" (id 2) (at 120.904 105.9688 0)

Commit message: Fixed value label of inductor
Parts:
- renumbered C3 to C12, C4 to C13, C5 to C14, C6 to C15, C7 to C16, U2 to U11
Changed lines of the file:
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@@
   (symbol (lib_id "power:GND") (at 142.748 116.586 0) (unit 1)
     (in_bom yes) (on_board yes) (fields_autoplaced)
-    (property "Reference" "#PWR012" (id 0) (at 142.748 122.936 0)
+    (property "Reference" "#PWR056" (id 0) (at 142.748 122.936 0)
       (effects (font (size 1.27 1.27)) hide)
     )
@@
   (symbol (lib_id "Device:C") (at 105.41 72.136 0) (unit 1)
     (in_bom yes) (on_board yes)
-    (property "Reference" "C3" (id 0) (at 109.474 70.8659 0)
+    (property "Reference" "C12" (id 0) (at 109.474 70.8659 0)
       (effects (font (size 1.27 1.27)) (justify left))
     )
@@
   (symbol (lib_id "Device:C") (at 179.324 106.934 90) (unit 1)
     (in_bom yes) (on_board yes)
-    (property "Reference" "C7" (id 0) (at 179.324 99.06 90))
+    (property "Reference" "C16" (id 0) (at 179.324 99.06 90))
     (property "Value" "1n" (id 1) (at 179.324 101.6 90))
     (property "Footprint" "Capacitor_SMD:C_0402_1005Metric" (id 2) (at 183.134 105.9688 0)
@@
   (symbol (lib_id "Device:C") (at 177.546 85.09 180) (unit 1)
     (in_bom yes) (on_board yes)
-    (property "Reference" "C6" (id 0) (at 173.482 86.3601 0)
+    (property "Reference" "C15" (id 0) (at 173.482 86.3601 0)
       (effects (font (size 1.27 1.27)) (justify left))
     )
@@
   (symbol (lib_id "Device:C") (at 130.048 72.136 0) (unit 1)
     (in_bom yes) (on_board yes)
-    (property "Reference" "C5" (id 0) (at 134.112 70.8659 0)
+    (property "Reference" "C14" (id 0) (at 134.112 70.8659 0)
       (effects (font (size 1.27 1.27)) (justify left))
     )
@@
   (symbol (lib_id "power:GND") (at 177.546 88.9 0) (unit 1)
     (in_bom yes) (on_board yes) (fields_autoplaced)
-    (property "Reference" "#PWR013" (id 0) (at 177.546 95.25 0)
+    (property "Reference" "#PWR057" (id 0) (at 177.546 95.25 0)
       (effects (font (size 1.27 1.27)) hide)
     )
@@
   (symbol (lib_id "power:GND") (at 105.41 75.946 0) (unit 1)
     (in_bom yes) (on_board yes) (fields_autoplaced)
-    (property "Reference" "#PWR010" (id 0) (at 105.41 82.296 0)
+    (property "Reference" "#PWR054" (id 0) (at 105.41 82.296 0)
       (effects (font (size 1.27 1.27)) hide)
     )
@@
   (symbol (lib_id "power:GND") (at 130.048 75.946 0) (unit 1)
     (in_bom yes) (on_board yes) (fields_autoplaced)
-    (property "Reference" "#PWR011" (id 0) (at 130.048 82.296 0)
+    (property "Reference" "#PWR055" (id 0) (at 130.048 82.296 0)
       (effects (font (size 1.27 1.27)) hide)
     )
@@
   (symbol (lib_id "Chubut2:PSA4-5043+") (at 142.748 103.124 0) (unit 1)
     (in_bom yes) (on_board yes) (fields_autoplaced)
-    (property "Reference" "U2" (id 0) (at 142.748 99.06 0))
+    (property "Reference" "U11" (id 0) (at 142.748 99.06 0))
     (property "Value" "PSA4-5043+" (id 1) (at 142.748 101.6 0))
     (property "Footprint" "chubut:MMM1362" (id 2) (at 142.748 103.124 0)
@@
   (symbol (lib_id "Device:C") (at 117.094 106.934 90) (unit 1)
     (in_bom yes) (on_board yes)
-    (property "Reference" "C4" (id 0) (at 117.094 99.06 90))
+    (property "Reference" "C13" (id 0) (at 117.094 99.06 90))
     (property "Value" "1n" (id 1) (at 117.094 101.6 90))
     (property "Footprint" "Capacitor_SMD:C_0402_1005Metric" (id 2) (at 120.904 105.9688 0)
