File: Chubut_2/dc_power.kicad_sch (KiCad schematic)
At the start: 4 parts, among them J19 3-5V

Commit message: Minor fixes
Parts:
- renumbered J19 to J10
Changed lines of the file:
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@@
   (symbol (lib_id "Connector:Conn_Coaxial_Power") (at 113.792 116.078 0) (unit 1)
     (in_bom yes) (on_board yes) (fields_autoplaced)
-    (property "Reference" "J19" (id 0) (at 116.84 116.3319 0)
+    (property "Reference" "J10" (id 0) (at 116.84 116.3319 0)
       (effects (font (size 1.27 1.27)) (justify left))
     )
@@
   (symbol (lib_id "power:GND") (at 113.792 121.158 0) (unit 1)
     (in_bom yes) (on_board yes) (fields_autoplaced)
-    (property "Reference" "#PWR058" (id 0) (at 113.792 127.508 0)
+    (property "Reference" "#PWR033" (id 0) (at 113.792 127.508 0)
       (effects (font (size 1.27 1.27)) hide)
     )
