File: Chubut_2/double_stage_channel.kicad_sch (KiCad schematic)
At the start: 8 parts, among them J13 In, J14 Conn_01x01_Female, J15 Out

Commit message: Minor fixes
Parts:
- renumbered J13 to J4, J14 to J5, J15 to J6, JP3 to JP1, R9 to R1, R10 to R2, R11 to R3, R12 to R4
Other:
- note added: "This line is just in case the 2 stages don't work"
Changed lines of the file:
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@@
     (stroke (width 0) (type default) (color 0 0 0 0))
+  )
+  (text "This line is just in case the 2 stages don't work" (at 206.756 86.36 0)
+    (effects (font (size 1.27 1.27)) (justify left bottom))
   )
   (hierarchical_label "3-5V" (shape input) (at 150.876 89.154 180)
@@
   (symbol (lib_id "Connector:Conn_01x01_Male") (at 134.874 100.584 0) (unit 1)
     (in_bom yes) (on_board yes) (fields_autoplaced)
-    (property "Reference" "J13" (id 0) (at 135.509 95.25 0))
+    (property "Reference" "J4" (id 0) (at 135.509 95.25 0))
     (property "Value" "In" (id 1) (at 135.509 97.79 0))
     (property "Footprint" "chubut:MILL-MAX_0965-0-15-20-80-14-11-0" (id 2) (at 134.874 100.584 0)
@@
   (symbol (lib_id "Connector:Conn_Coaxial") (at 254.254 99.06 0) (unit 1)
     (in_bom yes) (on_board yes) (fields_autoplaced)
-    (property "Reference" "J15" (id 0) (at 257.556 98.0831 0)
+    (property "Reference" "J6" (id 0) (at 257.556 98.0831 0)
       (effects (font (size 1.27 1.27)) (justify left))
     )
@@
   (symbol (lib_id "Device:R") (at 147.32 114.3 0) (unit 1)
     (in_bom yes) (on_board yes) (fields_autoplaced)
-    (property "Reference" "R9" (id 0) (at 149.352 113.0299 0)
+    (property "Reference" "R1" (id 0) (at 149.352 113.0299 0)
       (effects (font (size 1.27 1.27)) (justify left))
     )
@@
   (symbol (lib_id "Connector:Conn_01x01_Female") (at 254.254 95.758 270) (unit 1)
     (in_bom yes) (on_board yes) (fields_autoplaced)
-    (property "Reference" "J14" (id 0) (at 255.778 93.8529 90)
+    (property "Reference" "J5" (id 0) (at 255.778 93.8529 90)
       (effects (font (size 1.27 1.27)) (justify left))
     )
@@
   (symbol (lib_id "Device:R") (at 196.088 103.632 180) (unit 1)
     (in_bom yes) (on_board yes) (fields_autoplaced)
-    (property "Reference" "R11" (id 0) (at 198.882 102.3619 0)
+    (property "Reference" "R3" (id 0) (at 198.882 102.3619 0)
       (effects (font (size 1.27 1.27)) (justify right))
     )
@@
   (symbol (lib_id "Device:R") (at 189.992 99.822 90) (unit 1)
     (in_bom yes) (on_board yes) (fields_autoplaced)
-    (property "Reference" "R10" (id 0) (at 189.992 93.726 90))
+    (property "Reference" "R2" (id 0) (at 189.992 93.726 90))
     (property "Value" "Ra" (id 1) (at 189.992 96.266 90))
     (property "Footprint" "Resistor_SMD:R_0402_1005Metric" (id 2) (at 189.992 101.6 90)
@@
   (symbol (lib_id "Device:R") (at 201.93 99.822 90) (unit 1)
     (in_bom yes) (on_board yes) (fields_autoplaced)
-    (property "Reference" "R12" (id 0) (at 201.93 93.726 90))
+    (property "Reference" "R4" (id 0) (at 201.93 93.726 90))
     (property "Value" "Ra" (id 1) (at 201.93 96.266 90))
     (property "Footprint" "Resistor_SMD:R_0402_1005Metric" (id 2) (at 201.93 101.6 90)
@@
   (symbol (lib_id "power:GND") (at 147.32 118.11 0) (unit 1)
     (in_bom yes) (on_board yes) (fields_autoplaced)
-    (property "Reference" "#PWR052" (id 0) (at 147.32 124.46 0)
+    (property "Reference" "#PWR011" (id 0) (at 147.32 124.46 0)
       (effects (font (size 1.27 1.27)) hide)
     )
@@
   (symbol (lib_id "power:GND") (at 196.088 107.442 0) (unit 1)
     (in_bom yes) (on_board yes) (fields_autoplaced)
-    (property "Reference" "#PWR053" (id 0) (at 196.088 113.792 0)
+    (property "Reference" "#PWR012" (id 0) (at 196.088 113.792 0)
       (effects (font (size 1.27 1.27)) hide)
     )
@@
   (symbol (lib_id "power:GND") (at 254.254 104.14 0) (unit 1)
     (in_bom yes) (on_board yes) (fields_autoplaced)
-    (property "Reference" "#PWR054" (id 0) (at 254.254 110.49 0)
+    (property "Reference" "#PWR013" (id 0) (at 254.254 110.49 0)
       (effects (font (size 1.27 1.27)) hide)
     )
@@
   (symbol (lib_id "Jumper:SolderJumper_2_Open") (at 194.564 86.868 0) (unit 1)
     (in_bom yes) (on_board yes) (fields_autoplaced)
-    (property "Reference" "JP3" (id 0) (at 194.564 81.28 0))
+    (property "Reference" "JP1" (id 0) (at 194.564 81.28 0))
     (property "Value" "SolderJumper_2_Open" (id 1) (at 194.564 83.82 0))
     (property "Footprint" "Jumper:SolderJumper-2_P1.3mm_Open_RoundedPad1.0x1.5mm" (id 2) (at 194.564 86.868 0)

Commit message: New version with shieldings and the other suggestions from the workshop
Parts:
- removed J5: Conn_01x01_Female, chubut:just_a_pad, symbol Connector:Conn_01x01_Female
- removed JP1: SolderJumper_2_Open, Jumper:SolderJumper-2_P1.3mm_Open_RoundedPad1.0x1.5mm, symbol Jumper:SolderJumper_2_Open
- removed R2, R4: Ra, Resistor_SMD:R_0402_1005Metric, symbol Device:R
- removed R3: Rb, Resistor_SMD:R_0402_1005Metric, symbol Device:R
- renumbered J4 to J7, J6 to J8
Other:
- note removed: "This line is just in case the 2 stages don't work"
Changed lines of the file:
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@@
   (junction (at 154.94 105.918) (diameter 0) (color 0 0 0 0)
   )
-  (junction (at 183.642 99.822) (diameter 0) (color 0 0 0 0)
-  )
-  (junction (at 196.088 99.822) (diameter 0) (color 0 0 0 0)
-  )
   (wire (pts (xy 139.954 100.584) (xy 147.32 100.584))
-    (stroke (width 0) (type default) (color 0 0 0 0))
-  )
-  (wire (pts (xy 193.802 99.822) (xy 196.088 99.822))
-    (stroke (width 0) (type default) (color 0 0 0 0))
-  )
-  (wire (pts (xy 183.642 99.822) (xy 186.182 99.822))
-    (stroke (width 0) (type default) (color 0 0 0 0))
-  )
-  (wire (pts (xy 190.754 86.868) (xy 183.642 86.868))
-    (stroke (width 0) (type default) (color 0 0 0 0))
-  )
-  (wire (pts (xy 254.254 86.868) (xy 254.254 90.678))
     (stroke (width 0) (type default) (color 0 0 0 0))
   )
@@
     (stroke (width 0) (type default) (color 0 0 0 0))
   )
-  (wire (pts (xy 196.088 99.822) (xy 198.12 99.822))
-    (stroke (width 0) (type default) (color 0 0 0 0))
-  )
   (wire (pts (xy 147.32 100.584) (xy 147.32 110.49))
-    (stroke (width 0) (type default) (color 0 0 0 0))
-  )
-  (wire (pts (xy 198.374 86.868) (xy 254.254 86.868))
     (stroke (width 0) (type default) (color 0 0 0 0))
   )
@@
     (stroke (width 0) (type default) (color 0 0 0 0))
   )
-  (wire (pts (xy 183.642 86.868) (xy 183.642 99.822))
-    (stroke (width 0) (type default) (color 0 0 0 0))
-  )
-  (wire (pts (xy 205.74 99.822) (xy 214.63 99.822))
-    (stroke (width 0) (type default) (color 0 0 0 0))
-  )
-  (wire (pts (xy 180.34 99.822) (xy 183.642 99.822))
+  (wire (pts (xy 180.34 99.822) (xy 214.63 99.822))
     (stroke (width 0) (type default) (color 0 0 0 0))
   )
@@
     (stroke (width 0) (type default) (color 0 0 0 0))
   )
-  (text "This line is just in case the 2 stages don't work" (at 206.756 86.36 0)
-    (effects (font (size 1.27 1.27)) (justify left bottom))
-  )
   (hierarchical_label "3-5V" (shape input) (at 150.876 89.154 180)
     (effects (font (size 1.27 1.27)) (justify right))
@@
   (symbol (lib_id "Connector:Conn_01x01_Male") (at 134.874 100.584 0) (unit 1)
     (in_bom yes) (on_board yes) (fields_autoplaced)
-    (property "Reference" "J4" (id 0) (at 135.509 95.25 0))
+    (property "Reference" "J7" (id 0) (at 135.509 95.25 0))
     (property "Value" "In" (id 1) (at 135.509 97.79 0))
     (property "Footprint" "chubut:MILL-MAX_0965-0-15-20-80-14-11-0" (id 2) (at 134.874 100.584 0)
@@
   (symbol (lib_id "Connector:Conn_Coaxial") (at 254.254 99.06 0) (unit 1)
     (in_bom yes) (on_board yes) (fields_autoplaced)
-    (property "Reference" "J6" (id 0) (at 257.556 98.0831 0)
+    (property "Reference" "J8" (id 0) (at 257.556 98.0831 0)
       (effects (font (size 1.27 1.27)) (justify left))
     )
@@
     (pin "2")
   )
-  (symbol (lib_id "Connector:Conn_01x01_Female") (at 254.254 95.758 270) (unit 1)
-    (in_bom yes) (on_board yes) (fields_autoplaced)
-    (property "Reference" "J5" (id 0) (at 255.778 93.8529 90)
-      (effects (font (size 1.27 1.27)) (justify left))
-    )
-    (property "Value" "Conn_01x01_Female" (id 1) (at 255.778 96.3929 90)
-      (effects (font (size 1.27 1.27)) (justify left))
-    )
-    (property "Footprint" "chubut:just_a_pad" (id 2) (at 254.254 95.758 0)
-      (effects (font (size 1.27 1.27)) hide)
-    )
-    (property "Datasheet" "~" (id 3) (at 254.254 95.758 0)
-      (effects (font (size 1.27 1.27)) hide)
-    )
-    (pin "1")
-  )
-  (symbol (lib_id "Device:R") (at 196.088 103.632 180) (unit 1)
-    (in_bom yes) (on_board yes) (fields_autoplaced)
-    (property "Reference" "R3" (id 0) (at 198.882 102.3619 0)
-      (effects (font (size 1.27 1.27)) (justify right))
-    )
-    (property "Value" "Rb" (id 1) (at 198.882 104.9019 0)
-      (effects (font (size 1.27 1.27)) (justify right))
-    )
-    (property "Footprint" "Resistor_SMD:R_0402_1005Metric" (id 2) (at 197.866 103.632 90)
-      (effects (font (size 1.27 1.27)) hide)
-    )
-    (property "Datasheet" "~" (id 3) (at 196.088 103.632 0)
-      (effects (font (size 1.27 1.27)) hide)
-    )
-    (pin "1")
-    (pin "2")
-  )
-  (symbol (lib_id "Device:R") (at 189.992 99.822 90) (unit 1)
-    (in_bom yes) (on_board yes) (fields_autoplaced)
-    (property "Reference" "R2" (id 0) (at 189.992 93.726 90))
-    (property "Value" "Ra" (id 1) (at 189.992 96.266 90))
-    (property "Footprint" "Resistor_SMD:R_0402_1005Metric" (id 2) (at 189.992 101.6 90)
-      (effects (font (size 1.27 1.27)) hide)
-    )
-    (property "Datasheet" "~" (id 3) (at 189.992 99.822 0)
-      (effects (font (size 1.27 1.27)) hide)
-    )
-    (pin "1")
-    (pin "2")
-  )
-  (symbol (lib_id "Device:R") (at 201.93 99.822 90) (unit 1)
-    (in_bom yes) (on_board yes) (fields_autoplaced)
-    (property "Reference" "R4" (id 0) (at 201.93 93.726 90))
-    (property "Value" "Ra" (id 1) (at 201.93 96.266 90))
-    (property "Footprint" "Resistor_SMD:R_0402_1005Metric" (id 2) (at 201.93 101.6 90)
-      (effects (font (size 1.27 1.27)) hide)
-    )
-    (property "Datasheet" "~" (id 3) (at 201.93 99.822 0)
-      (effects (font (size 1.27 1.27)) hide)
-    )
-    (pin "1")
-    (pin "2")
-  )
   (symbol (lib_id "power:GND") (at 147.32 118.11 0) (unit 1)
     (in_bom yes) (on_board yes) (fields_autoplaced)
-    (property "Reference" "#PWR011" (id 0) (at 147.32 124.46 0)
+    (property "Reference" "#PWR014" (id 0) (at 147.32 124.46 0)
       (effects (font (size 1.27 1.27)) hide)
     )
@@
     (pin "1")
   )
-  (symbol (lib_id "power:GND") (at 196.088 107.442 0) (unit 1)
-    (in_bom yes) (on_board yes) (fields_autoplaced)
-    (property "Reference" "#PWR012" (id 0) (at 196.088 113.792 0)
-      (effects (font (size 1.27 1.27)) hide)
-    )
-    (property "Value" "GND" (id 1) (at 196.088 112.776 0))
-    (property "Footprint" "" (id 2) (at 196.088 107.442 0)
-      (effects (font (size 1.27 1.27)) hide)
-    )
-    (property "Datasheet" "" (id 3) (at 196.088 107.442 0)
-      (effects (font (size 1.27 1.27)) hide)
-    )
-    (pin "1")
-  )
   (symbol (lib_id "power:GND") (at 254.254 104.14 0) (unit 1)
     (in_bom yes) (on_board yes) (fields_autoplaced)
-    (property "Reference" "#PWR013" (id 0) (at 254.254 110.49 0)
+    (property "Reference" "#PWR016" (id 0) (at 254.254 110.49 0)
       (effects (font (size 1.27 1.27)) hide)
     )
@@
     (pin "1")
   )
-  (symbol (lib_id "Jumper:SolderJumper_2_Open") (at 194.564 86.868 0) (unit 1)
-    (in_bom yes) (on_board yes) (fields_autoplaced)
-    (property "Reference" "JP1" (id 0) (at 194.564 81.28 0))
-    (property "Value" "SolderJumper_2_Open" (id 1) (at 194.564 83.82 0))
-    (property "Footprint" "Jumper:SolderJumper-2_P1.3mm_Open_RoundedPad1.0x1.5mm" (id 2) (at 194.564 86.868 0)
-      (effects (font (size 1.27 1.27)) hide)
-    )
-    (property "Datasheet" "~" (id 3) (at 194.564 86.868 0)
-      (effects (font (size 1.27 1.27)) hide)
-    )
-    (pin "1")
-    (pin "2")
-  )
   (sheet (at 157.734 95.25) (size 22.606 14.732) (fields_autoplaced)
