File: Chubut_2/temperature_and_humidity_sensor.kicad_sch (KiCad schematic)
At the start: 3 parts, among them J31 Conn_01x04, U13 SHT31-DIS

Commit message: Several updates
Parts:
- renumbered C19 to C22, J31 to J29
Changed lines of the file:
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@@
   (symbol (lib_id "Device:C") (at 117.602 107.696 0) (mirror y) (unit 1)
     (in_bom yes) (on_board yes)
-    (property "Reference" "C19" (id 0) (at 114.681 106.5276 0)
+    (property "Reference" "C22" (id 0) (at 114.681 106.5276 0)
       (effects (font (size 1.27 1.27)) (justify left))
     )
@@
   (symbol (lib_id "Connector_Generic:Conn_01x04") (at 155.448 107.696 0) (unit 1)
     (in_bom yes) (on_board yes)
-    (property "Reference" "J31" (id 0) (at 157.48 107.8992 0)
+    (property "Reference" "J29" (id 0) (at 157.48 107.8992 0)
       (effects (font (size 1.27 1.27)) (justify left))
     )

Commit message: First layout of second prototyping iteration
Parts:
- J5: renamed from J29; value Conn_01x04 -> T+H_sensor; footprint chubut:850-10-004-10-001101 -> Connector_JST:JST_XH_S4B-XH-A_1x04_P2.50mm_Horizontal; Digikey https://www.digikey.ch/short/m772hmt3 -> https://www.digikey.ch/de/products/detail/jst-sales-america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; Manufacturer Preci-Dip -> JST Sales America Inc.; Manufacturer number 850-10-004-10-001101 -> S4B-XH-A-1(LF)(SN)
- renumbered C22 to C9, U13 to U9
Changed lines of the file:
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@@
   (symbol (lib_id "Device:C") (at 117.602 107.696 0) (mirror y) (unit 1)
     (in_bom yes) (on_board yes)
-    (property "Reference" "C22" (id 0) (at 114.681 106.5276 0)
+    (property "Reference" "C9" (id 0) (at 114.681 106.5276 0)
       (effects (font (size 1.27 1.27)) (justify left))
     )
@@
   (symbol (lib_id "Sensor_Humidity:SHT31-DIS") (at 135.89 107.696 0) (unit 1)
     (in_bom yes) (on_board yes)
-    (property "Reference" "U13" (id 0) (at 135.89 95.4786 0))
+    (property "Reference" "U9" (id 0) (at 135.89 95.4786 0))
     (property "Value" "SHT31-DIS" (id 1) (at 135.89 97.79 0))
     (property "Footprint" "Sensor_Humidity:Sensirion_DFN-8-1EP_2.5x2.5mm_P0.5mm_EP1.1x1.7mm" (id 2) (at 135.89 106.426 0)
@@
   (symbol (lib_id "Connector_Generic:Conn_01x04") (at 155.448 107.696 0) (unit 1)
     (in_bom yes) (on_board yes)
-    (property "Reference" "J29" (id 0) (at 157.48 107.8992 0)
+    (property "Reference" "J5" (id 0) (at 157.48 107.8992 0)
       (effects (font (size 1.27 1.27)) (justify left))
     )
-    (property "Value" "Conn_01x04" (id 1) (at 157.48 110.2106 0)
+    (property "Value" "T+H_sensor" (id 1) (at 157.48 110.2106 0)
       (effects (font (size 1.27 1.27)) (justify left))
     )
-    (property "Footprint" "chubut:850-10-004-10-001101" (id 2) (at 155.448 107.696 0)
+    (property "Footprint" "Connector_JST:JST_XH_S4B-XH-A_1x04_P2.50mm_Horizontal" (id 2) (at 155.448 107.696 0)
       (effects (font (size 1.27 1.27)) hide)
     )
-    (property "Datasheet" "https://www.precidip.com/AppHost/9696,1/Scripts/Modules/Catalog/Default.aspx?c=8&i=520&p=171&pdf=1&dsku=850-PP-NNN-10-001101" (id 3) (at 155.448 107.696 0)
+    (property "Datasheet" "https://www.jst-mfg.com/product/pdf/eng/eXH.pdf" (id 3) (at 155.448 107.696 0)
       (effects (font (size 1.27 1.27)) hide)
     )
-    (property "Manufacturer number" "850-10-004-10-001101" (id 4) (at 170.688 112.776 0))
-    (property "Digikey" "https://www.digikey.ch/short/m772hmt3" (id 5) (at 155.448 107.696 0)
+    (property "Manufacturer number" "S4B-XH-A-1(LF)(SN)" (id 4) (at 168.148 112.776 0))
+    (property "Digikey" "https://www.digikey.ch/de/products/detail/jst-sales-america-inc/S4B-XH-A-1-LF-SN/9961923" (id 5) (at 155.448 107.696 0)
       (effects (font (size 1.27 1.27)) hide)
     )
-    (property "Manufacturer" "Preci-Dip" (id 6) (at 155.448 107.696 0)
+    (property "Manufacturer" "JST Sales America Inc." (id 6) (at 155.448 107.696 0)
       (effects (font (size 1.27 1.27)) hide)
     )

Commit message: Minor fixes
Parts:
- renumbered C9 to C5, J5 to J3, U9 to U5
Changed lines of the file:
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@@
   (symbol (lib_id "Device:C") (at 117.602 107.696 0) (mirror y) (unit 1)
     (in_bom yes) (on_board yes)
-    (property "Reference" "C9" (id 0) (at 114.681 106.5276 0)
+    (property "Reference" "C5" (id 0) (at 114.681 106.5276 0)
       (effects (font (size 1.27 1.27)) (justify left))
     )
@@
   (symbol (lib_id "Sensor_Humidity:SHT31-DIS") (at 135.89 107.696 0) (unit 1)
     (in_bom yes) (on_board yes)
-    (property "Reference" "U9" (id 0) (at 135.89 95.4786 0))
+    (property "Reference" "U5" (id 0) (at 135.89 95.4786 0))
     (property "Value" "SHT31-DIS" (id 1) (at 135.89 97.79 0))
     (property "Footprint" "Sensor_Humidity:Sensirion_DFN-8-1EP_2.5x2.5mm_P0.5mm_EP1.1x1.7mm" (id 2) (at 135.89 106.426 0)
@@
   (symbol (lib_id "Connector_Generic:Conn_01x04") (at 155.448 107.696 0) (unit 1)
     (in_bom yes) (on_board yes)
-    (property "Reference" "J5" (id 0) (at 157.48 107.8992 0)
+    (property "Reference" "J3" (id 0) (at 157.48 107.8992 0)
       (effects (font (size 1.27 1.27)) (justify left))
     )

Commit message: New version with shieldings and the other suggestions from the workshop
Parts:
- renumbered J3 to J6
Changed lines of the file:
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@@
   (symbol (lib_id "Connector_Generic:Conn_01x04") (at 155.448 107.696 0) (unit 1)
     (in_bom yes) (on_board yes)
-    (property "Reference" "J3" (id 0) (at 157.48 107.8992 0)
+    (property "Reference" "J6" (id 0) (at 157.48 107.8992 0)
       (effects (font (size 1.27 1.27)) (justify left))
     )
