File: Carrier_2/Carrier_2.kicad_pcb (KiCad board)
At the start: 4 copper layers, 18 x 32.8 mm, 21 parts, among them J1 HV, J2 3-5V, J3 Out 1, J4 Out 2, U1 LGAD_2_pad, U12 PSA4-5043+, U2 PSA4-5043+

Commit message: Several updates
Parts:
- removed C16: 1n, Capacitor_SMD:C_0402_1005Metric
- removed the C5 at (6.00, 3.30)
- added C11: 100p, Capacitor_SMD:C_0402_1005Metric, F.Cu at (6.00, 10.2)
- added C2: 820p, Capacitor_SMD:C_0805_2012Metric, F.Cu at (6.00, 3.50)
- added C6: 100p, Capacitor_SMD:C_0402_1005Metric, F.Cu at (-5.83, 9.51)
- added C7: 1n, Capacitor_SMD:C_0402_1005Metric, F.Cu at (-3.35, 9.61)
- added C8: 100p, Capacitor_SMD:C_0402_1005Metric, F.Cu at (7.51, 10.2)
- added C9: 1n, Capacitor_SMD:C_0402_1005Metric, F.Cu at (1.04, 5.21)
- C1: value 1n -> 820p; footprint Capacitor_SMD:C_0402_1005Metric -> Capacitor_SMD:C_0805_2012Metric
- C12: value ~ -> 1n
- C3: value ~ -> 100p
- C4: value 10n -> 1n; footprint Capacitor_SMD:C_0805_2012Metric -> Capacitor_SMD:C_0402_1005Metric
- moved C3 10.6 mm to (-7.36, 9.52)
- moved C1 7.22 mm to (-6.00, 3.50)
- moved C12 6.58 mm to (3.22, 10.1)
- moved C4 5.32 mm to (-1.05, 5.25)
- renumbered C2 to C10, C17 to C5, U12 to U2, U2 to U3
Connections:
- C1 pad 1: /Channel_2/In -> /HV
- C1 pad 2: Net-(C1-Pad2) -> GND
- C12 pad 2: /Channel_1/Out -> /Channel_2/Out
- C3 pad 1: Net-(C3-Pad1) -> /Channel_1/3-5V
- C3 pad 2: /Channel_2/Out -> GND
- C4 pad 1: /HV -> /Channel_1/In
- C4 pad 2: GND -> Net-(C4-Pad2)
- L2 pad 2: Net-(C12-Pad1) -> Net-(C7-Pad1)
- L4 pad 2: Net-(C3-Pad1) -> Net-(C12-Pad1)
- U2 pad 1: Net-(C12-Pad1) -> Net-(C7-Pad1)
- U2 pad 3: Net-(C16-Pad2) -> Net-(C4-Pad2)
- U3 pad 1: Net-(C3-Pad1) -> Net-(C12-Pad1)
- U3 pad 3: Net-(C1-Pad2) -> Net-(C9-Pad2)
Routing:
- net /Channel_1/3-5V: track 26.8 -> 30.9 mm, vias 2 -> 3
- net Net-(C3-Pad1): track 2.23 -> 0.00 mm
- net Net-(C7-Pad1): track 0.00 -> 2.15 mm
- net Net-(C9-Pad2): track 0.00 -> 1.64 mm
- net Net-(C1-Pad2): track 1.64 -> 0.00 mm
- net Net-(C6-Pad2): track 1.07 -> 2.18 mm
- net Net-(C11-Pad2): track 1.04 -> 2.12 mm
- net Net-(C4-Pad2): track 0.00 -> 1.04 mm
- net Net-(C16-Pad2): track 1.04 -> 0.00 mm
