File: Carrier_2/Carrier_2.kicad_pcb (KiCad board)
At the start: 4 copper layers, 18 x 32.8 mm, 25 parts, among them J1 HV, J2 3-5V, J3 Out 1, J4 Out 2, U1 LGAD_2_pad, U2 PSA4-5043+, U3 PSA4-5043+

Commit message: Removed silkscreen and fixed one track
Other:
- board text added: "Chubut 2, Carrier_2 220824"
Changed lines of the file:
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@@
   )
   (gr_rect (start -9 16.8) (end 9 -16) (layer "Edge.Cuts") (width 0.1) (fill none))
+  (gr_text "Chubut 2, Carrier_2\n220824" (at -8.42 -13.76) (layer "F.SilkS")
+    (effects (font (size 1 1) (thickness 0.15)) (justify left))
+  )
   (segment (start 1 4.74) (end 1.01 4.75) (width 0.25) (layer "F.Cu") (net 1))
   (segment (start 1 3) (end 1 4.74) (width 0.25) (layer "F.Cu") (net 1))

Commit message: Added value to 2 inductors that was missing and cleaned up the F.Fab
Parts:
- L1, L3: value L -> 1µ
- L2, L4: value L -> 18n
Changed lines of the file:
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@@
       (effects (font (size 1 1) (thickness 0.15)))
     )
-    (fp_text value "100n" (at 0 1.68) (layer "F.Fab")
+    (fp_text value "100n" (at 0 1.68) (layer "F.Fab") hide
       (effects (font (size 1 1) (thickness 0.15)))
     )
@@
       (effects (font (size 1 1) (thickness 0.15)))
     )
-    (fp_text value "100p" (at 0 1.16 90) (layer "F.Fab")
+    (fp_text value "100p" (at 0 1.16 90) (layer "F.Fab") hide
       (effects (font (size 1 1) (thickness 0.15)))
     )
@@
       (effects (font (size 1 1) (thickness 0.15)))
     )
-    (fp_text value "PSA4-5043+" (at 0.25 1.6 90 unlocked) (layer "F.Fab")
-      (effects (font (size 1 1) (thickness 0.15)))
-    )
-    (fp_text user "${REFERENCE}" (at 0.25 3.1 90 unlocked) (layer "F.Fab")
+    (fp_text value "PSA4-5043+" (at 0.25 1.6 90 unlocked) (layer "F.Fab") hide
+      (effects (font (size 1 1) (thickness 0.15)))
+    )
+    (fp_text user "${REFERENCE}" (at 0.25 3.1 90 unlocked) (layer "F.Fab") hide
       (effects (font (size 1 1) (thickness 0.15)))
     )
@@
       (effects (font (size 1 1) (thickness 0.15)))
     )
-    (fp_text value "1n" (at 0 1.16 90) (layer "F.Fab")
+    (fp_text value "1n" (at 0 1.16 90) (layer "F.Fab") hide
       (effects (font (size 1 1) (thickness 0.15)))
     )
@@
       (effects (font (size 1 1) (thickness 0.15)))
     )
-    (fp_text value "100p" (at 0 1.16 90) (layer "F.Fab")
+    (fp_text value "100p" (at 0 1.16 90) (layer "F.Fab") hide
       (effects (font (size 1 1) (thickness 0.15)))
     )
@@
       (effects (font (size 1 1) (thickness 0.15)))
     )
-    (fp_text value "100p" (at 0 1.16 90) (layer "F.Fab")
+    (fp_text value "100p" (at 0 1.16 90) (layer "F.Fab") hide
       (effects (font (size 1 1) (thickness 0.15)))
     )
@@
       (effects (font (size 1 1) (thickness 0.15)))
     )
-    (fp_text value "100n" (at 0 1.68) (layer "F.Fab")
+    (fp_text value "100n" (at 0 1.68) (layer "F.Fab") hide
       (effects (font (size 1 1) (thickness 0.15)))
     )
@@
       (effects (font (size 1 1) (thickness 0.15)))
     )
-    (fp_text value "LGAD_2_pad" (at 0 5.72 unlocked) (layer "F.Fab")
-      (effects (font (size 1 1) (thickness 0.15)))
-    )
-    (fp_text user "${REFERENCE}" (at 0 7.22 unlocked) (layer "F.Fab")
+    (fp_text value "LGAD_2_pad" (at 0 5.72 unlocked) (layer "F.Fab") hide
+      (effects (font (size 1 1) (thickness 0.15)))
+    )
+    (fp_text user "${REFERENCE}" (at 0 7.22 unlocked) (layer "F.Fab") hide
       (effects (font (size 1 1) (thickness 0.15)))
     )
@@
       (effects (font (size 1 1) (thickness 0.15)))
     )
-    (fp_text value "1n" (at 0 1.16 90) (layer "F.Fab")
+    (fp_text value "1n" (at 0 1.16 90) (layer "F.Fab") hide
       (effects (font (size 1 1) (thickness 0.15)))
     )
@@
       (effects (font (size 1 1) (thickness 0.15)))
     )
-    (fp_text value "1n" (at 0 1.16 90) (layer "F.Fab")
+    (fp_text value "1n" (at 0 1.16 90) (layer "F.Fab") hide
       (effects (font (size 1 1) (thickness 0.15)))
     )
@@
       (effects (font (size 1 1) (thickness 0.15)))
     )
-    (fp_text value "1n" (at 0 1.16 90) (layer "F.Fab")
+    (fp_text value "1n" (at 0 1.16 90) (layer "F.Fab") hide
       (effects (font (size 1 1) (thickness 0.15)))
     )
@@
       (effects (font (size 1 1) (thickness 0.15)))
     )
-    (fp_text value "L" (at 0 1.17) (layer "F.Fab")
+    (fp_text value "1µ" (at 0 1.17) (layer "F.Fab") hide
       (effects (font (size 1 1) (thickness 0.15)))
     )
@@
       (effects (font (size 1 1) (thickness 0.15)))
     )
-    (fp_text value "L" (at 0 1.17) (layer "F.Fab")
+    (fp_text value "1µ" (at 0 1.17) (layer "F.Fab") hide
       (effects (font (size 1 1) (thickness 0.15)))
     )
@@
       (effects (font (size 1 1) (thickness 0.15)))
     )
-    (fp_text value "10k" (at 0 1.17 90) (layer "F.Fab")
+    (fp_text value "10k" (at 0 1.17 90) (layer "F.Fab") hide
       (effects (font (size 1 1) (thickness 0.15)))
     )
@@
       (effects (font (size 1 1) (thickness 0.15)))
     )
-    (fp_text value "3-5V" (at 0 -2.2 180 unlocked) (layer "F.Fab")
-      (effects (font (size 1 1) (thickness 0.15)))
-    )
-    (fp_text user "${REFERENCE}" (at 0 -0.7 180 unlocked) (layer "F.Fab")
+    (fp_text value "3-5V" (at 0 -2.2 unlocked) (layer "F.Fab")
+      (effects (font (size 1 1) (thickness 0.15)))
+    )
+    (fp_text user "${REFERENCE}" (at 0 -0.7 unlocked) (layer "F.Fab")
       (effects (font (size 1 1) (thickness 0.15)))
     )
@@
       (effects (font (size 1 1) (thickness 0.15)))
     )
-    (fp_text value "Out 1" (at 0 -2.2 180 unlocked) (layer "F.Fab")
-      (effects (font (size 1 1) (thickness 0.15)))
-    )
-    (fp_text user "${REFERENCE}" (at 0 -0.7 180 unlocked) (layer "F.Fab")
+    (fp_text value "Out 1" (at 0 -2.2 unlocked) (layer "F.Fab")
+      (effects (font (size 1 1) (thickness 0.15)))
+    )
+    (fp_text user "${REFERENCE}" (at 0 -0.7 unlocked) (layer "F.Fab")
       (effects (font (size 1 1) (thickness 0.15)))
     )
@@
       (effects (font (size 1 1) (thickness 0.15)))
     )
-    (fp_text value "PSA4-5043+" (at 0.25 1.6 unlocked) (layer "F.Fab")
-      (effects (font (size 1 1) (thickness 0.15)))
-    )
-    (fp_text user "${REFERENCE}" (at 0.25 3.1 unlocked) (layer "F.Fab")
+    (fp_text value "PSA4-5043+" (at 0.25 1.6 unlocked) (layer "F.Fab") hide
+      (effects (font (size 1 1) (thickness 0.15)))
+    )
+    (fp_text user "${REFERENCE}" (at 0.25 3.1 unlocked) (layer "F.Fab") hide
       (effects (font (size 1 1) (thickness 0.15)))
     )
@@
       (effects (font (size 1 1) (thickness 0.15)))
     )
-    (fp_text value "HV" (at 0 -2.2 180 unlocked) (layer "F.Fab")
-      (effects (font (size 1 1) (thickness 0.15)))
-    )
-    (fp_text user "${REFERENCE}" (at 0 -0.7 180 unlocked) (layer "F.Fab")
+    (fp_text value "HV" (at 0 -2.2 unlocked) (layer "F.Fab")
+      (effects (font (size 1 1) (thickness 0.15)))
+    )
+    (fp_text user "${REFERENCE}" (at 0 -0.7 unlocked) (layer "F.Fab")
       (effects (font (size 1 1) (thickness 0.15)))
     )
@@
       (effects (font (size 1 1) (thickness 0.15)))
     )
-    (fp_text value "10k" (at 0 1.17 90) (layer "F.Fab")
+    (fp_text value "10k" (at 0 1.17 90) (layer "F.Fab") hide
       (effects (font (size 1 1) (thickness 0.15)))
     )
@@
       (effects (font (size 1 1) (thickness 0.15)))
     )
-    (fp_text value "820p" (at 0 1.68 90) (layer "F.Fab")
+    (fp_text value "820p" (at 0 1.68 90) (layer "F.Fab") hide
       (effects (font (size 1 1) (thickness 0.15)))
     )
@@
       (effects (font (size 1 1) (thickness 0.15)))
     )
-    (fp_text value "820p" (at 0 1.68 90) (layer "F.Fab")
+    (fp_text value "820p" (at 0 1.68 90) (layer "F.Fab") hide
       (effects (font (size 1 1) (thickness 0.15)))
     )
@@
       (effects (font (size 1 1) (thickness 0.15)))
     )
-    (fp_text value "Out 2" (at 0 -2.2 180 unlocked) (layer "F.Fab")
-      (effects (font (size 1 1) (thickness 0.15)))
-    )
-    (fp_text user "${REFERENCE}" (at 0 -0.7 180 unlocked) (layer "F.Fab")
+    (fp_text value "Out 2" (at 0 -2.2 unlocked) (layer "F.Fab")
+      (effects (font (size 1 1) (thickness 0.15)))
+    )
+    (fp_text user "${REFERENCE}" (at 0 -0.7 unlocked) (layer "F.Fab")
       (effects (font (size 1 1) (thickness 0.15)))
     )
@@
       (effects (font (size 1 1) (thickness 0.15)))
     )
-    (fp_text value "L" (at 0 1.17) (layer "F.Fab")
+    (fp_text value "18n" (at 0 1.17) (layer "F.Fab") hide
       (effects (font (size 1 1) (thickness 0.15)))
     )
@@
       (effects (font (size 1 1) (thickness 0.15)))
     )
-    (fp_text value "100p" (at 0 1.16 90) (layer "F.Fab")
+    (fp_text value "100p" (at 0 1.16 90) (layer "F.Fab") hide
       (effects (font (size 1 1) (thickness 0.15)))
     )
@@
       (effects (font (size 1 1) (thickness 0.15)))
     )
-    (fp_text value "L" (at 0 1.17) (layer "F.Fab")
-      (effects (font (size 1 1) (thickness 0.15)))
-    )
+    (fp_text value "18n" (at 0 1.17) (layer "F.Fab") hide
+      (effects (font (size 1 1) (thickness 0.15)))
+    )
