File: carrier_boards/RD50_TI-LGAD_P250_4x4/RD50_TI-LGAD_P250_4x4.kicad_pcb (KiCad board)
At the start: 2 copper layers, 39 x 10 mm, 11 parts, among them J10 CH1, J11 CH1, J12 CH1, J13 CH1, J14 CH1, J7 CH1, J9 HV, U1 LGAD_4CH_dual

Commit message: Improved routing by removing a via in the high voltage pad
Routing:
- net Net-(J9-Pin_1): track 11.3 -> 13.1 mm
Changed lines of the file:
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@@
   (segment (start -2.8 -1.3) (end -3.5 -2) (width 0.25) (layer "B.Cu") (net 4))
   (segment (start -2.72 -1.3) (end -2.8 -1.3) (width 0.25) (layer "B.Cu") (net 4))
-  (via (at -0.9005 -0.715907) (size 0.8) (drill 0.4) (layers "F.Cu" "B.Cu") (net 5))
-  (segment (start -1.634093 -0.715907) (end -0.9005 -0.715907) (width 0.25) (layer "B.Cu") (net 5))
-  (segment (start -7.68 2.32) (end -4.67 2.32) (width 0.25) (layer "B.Cu") (net 5))
-  (segment (start -4.67 2.32) (end -1.634093 -0.715907) (width 0.25) (layer "B.Cu") (net 5))
-  (segment (start -10 0) (end -7.68 2.32) (width 0.25) (layer "B.Cu") (net 5))
+  (segment (start -3.943173 -3.88) (end -0.614949 -0.551776) (width 0.25) (layer "F.Cu") (net 5))
+  (segment (start -0.614949 -0.551776) (end -0.583363 -0.583362) (width 0.25) (layer "F.Cu") (net 5))
+  (segment (start -8.78 -2.37) (end -7.27 -3.88) (width 0.25) (layer "F.Cu") (net 5))
+  (segment (start -7.27 -3.88) (end -3.943173 -3.88) (width 0.25) (layer "F.Cu") (net 5))
+  (via (at -8.78 -2.37) (size 0.8) (drill 0.4) (layers "F.Cu" "B.Cu") (net 5))
+  (segment (start -10 0) (end -10 -1.15) (width 0.25) (layer "B.Cu") (net 5))
+  (segment (start -10 -1.15) (end -8.78 -2.37) (width 0.25) (layer "B.Cu") (net 5))
   (via (at -0.27 2.71) (size 0.8) (drill 0.4) (layers "F.Cu" "B.Cu") (free) (net 6))
   (via (at -0.27 -2.93) (size 0.8) (drill 0.4) (layers "F.Cu" "B.Cu") (free) (net 6))

Commit message: Final improvements on the carrier before submision
Connections:
- net Net-(J9-Pin_1) renamed /HV
Routing:
- net /HV: track 13.1 -> 11.6 mm
Other:
- board text added: "${board_name}"
- board text added: "${timestamp}"
- board text added: "M. Senger"
- board text added: "UZH"
