File: carrier_boards/RD50_TI-LGAD_P250_4x4/RD50_TI-LGAD_P250_4x4.kicad_sch (KiCad schematic)
At the start: 11 parts, among them J10 CH1, J11 CH1, J12 CH1, J13 CH1, J14 CH1, J7 CH1, J9 HV, U1 LGAD_4CH_dual

Commit message: Final improvements on the carrier before submision
Connections:
- net HV: now reaches J9.1 (Pin_1), U1.1
Changed lines of the file:
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@@
     (stroke (width 0) (type default))
+  )
+  (label "HV" (at 113.03 132.08 0) (fields_autoplaced)
+    (effects (font (size 1.27 1.27)) (justify left bottom))
   )
   (symbol (lib_id "Mechanical:MountingHole") (at 130.81 106.68 0) (unit 1)
